File: Low_Bandpass_Filter/LBP.kicad_sch (KiCad schematic)
At the start: 28 parts, among them U1 OPA1641, U2 OPA1641, U3 OPA1641, U4 OPA1641

Commit message: finalised LBPF+changed names of files
Parts:
- C5, C7: value C -> 10u
- R1: value R -> 1k; footprint (none) -> Resistor_THT:R_Axial_DIN0207_L6.3mm_D2.5mm_P10.16mm_Horizontal
- R10, R9: value R -> 2k2; footprint (none) -> Resistor_THT:R_Axial_DIN0207_L6.3mm_D2.5mm_P10.16mm_Horizontal
- R11: value R -> 100k; footprint (none) -> Resistor_THT:R_Axial_DIN0207_L6.3mm_D2.5mm_P10.16mm_Horizontal
- R12, R13, R3, R4, R5, R6: value R -> 22k; footprint (none) -> Resistor_THT:R_Axial_DIN0207_L6.3mm_D2.5mm_P10.16mm_Horizontal
- R14: value R -> 100; footprint (none) -> Resistor_THT:R_Axial_DIN0207_L6.3mm_D2.5mm_P10.16mm_Horizontal
- R2: value R -> 3k3; footprint (none) -> Resistor_THT:R_Axial_DIN0207_L6.3mm_D2.5mm_P10.16mm_Horizontal
- R7, R8: value R -> 10k; footprint (none) -> Resistor_THT:R_Axial_DIN0207_L6.3mm_D2.5mm_P10.16mm_Horizontal
- RV3, RV4: value R_Potentiometer -> 10k
Connections:
- net at C4.1, U3.2 (-): now also R8.1; no longer R8.2
- net at C1.2, C5.2, RV1.4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: now also R5.2; no longer R5.1
- net at RV1.5: now also R8.2; no longer R8.1
- net at RV1.2: now also R7.2; no longer R7.1
- net at C1.1, U2.2 (-): now also R7.1; no longer R7.2
- net at R6.1, RV3.1, U1.3 (+): now also R5.1; no longer R5.2
Other:
- moved on the sheet: C5, R6

Commit message: few mods
changed 4 single op amps to 1 big 4 op amp
Parts:
- removed U1, U2, U3, U4: OPA1641, symbol Amplifier_Operational:OPA1641
- added IC1: OPA1644AIPWR, SOP65P640X120-14N, symbol OPA1644AIPWR:OPA1644AIPWR
- C1, C4: value C -> 12.7nF
- C2, C3: value C -> 100uF
- RV1: value ~ -> 10k
Connections:
- net +15V: now also IC1.4 (V+)
- net -15V: now also IC1.11 (V-)
- net GND: now also IC1.6 (-IN_B), IC1.9 (-IN_C)
- net C-: now reaches C4.1, R8.1
- net C-: now also IC1.10 (+IN_C)
- net Co: now reaches C4.2, R4.1
- net Co: now also IC1.8 (OUT_C)
- net Bo: now reaches C1.2, C5.2, R5.2, RV1.4
- net Bo: now also IC1.7 (OUT_B)
- net Ao: now reaches R3.1, RV1.1
- net Ao: now also IC1.1 (OUT_A)
- net A-: now reaches R2.1, R3.2, R4.2
- net A-: now also IC1.2 (-IN_A)
- net A+: now reaches R5.1, R6.1, RV3.1
- net A+: now also IC1.3 (+IN_A)
- net Do: now reaches C7.2, R12.2, RV4.3
- net Do: now also IC1.14 (OUT_D)
- net B-: now reaches C1.1, R7.1
- net B-: now also IC1.5 (+IN_B)
- net D+: now reaches C5.1, R11.1
- net D+: now also IC1.12 (+IN_D)
- net D-: now reaches R12.1, R13.2
- net D-: now also IC1.13 (-IN_D)
Other:
- moved on the sheet: R6, RV4

Commit message: simulated low bandpass
Parts:
- added R15, R18, R19, R22: 10k, Resistor_THT:R_Axial_DIN0207_L6.3mm_D2.5mm_P10.16mm_Horizontal, symbol Device:R
- added R16, R17, R20, R21: 10, Resistor_THT:R_Axial_DIN0207_L6.3mm_D2.5mm_P10.16mm_Horizontal, symbol Device:R
- added U1, U2, U3, U4: OPA1641, OPA1641:OPA1641, symbol Amplifier_Operational:OPA1641
- added V1, V2: 16, symbol Simulation_SPICE:VDC
- added V3: VSIN, symbol Simulation_SPICE:VSIN
- C6: value C -> 10u
Connections:
- net A+: no longer R5.1, R6.1, RV3.1
- net A-: no longer R2.1, R3.2, R4.2
- net Ao: no longer R3.1, RV1.1
- net B-: no longer C1.1, R7.1
- net Bo: no longer C1.2, C5.2, R5.2, RV1.4
- net C-: no longer C4.1, R8.1
- net Co: no longer C4.2, R4.1
- net D+: no longer C5.1, R11.1
- net D-: no longer R12.1, R13.2
- net Do: no longer C7.2, R12.2, RV4.3
- net Input: now also V3.1
- net at C6.1, R13.1: now also R21.2; no longer RV4.1
- net at RV1.5: no longer R8.2
- net at RV1.6: no longer R10.1
- net at RV1.2: no longer R7.2
- net at RV1.3: no longer R9.1
- net at R1.1: now also R15.1, R16.2; no longer RV3.2
- net at R2.2: now also R15.2; no longer RV3.3
- net at R6.2: now also R21.1, R22.2; no longer RV4.2
- net +15V: no longer names the net of IC1.4 (V+)
- net -15V: no longer names the net of IC1.11 (V-)
- net GND renamed 0
- net 0: now also U1.3 (+), U2.3 (+), V1.1, V2.2, V3.2; no longer IC1.6 (-IN_B), IC1.9 (-IN_C)
- new net: C4.1, R8.1, U2.2 (-)
- new net: C4.2, R4.1, U2.6
- new net: R2.1, R3.2, R4.2, U3.2 (-)
- new net: R16.1, R5.1, R6.1, U3.3 (+)
- new net: R18.2, R3.1, U3.6
- new net: C7.2, R12.2, R22.1, U4.6
- new net: R10.1, R20.1
- new net: C1.1, R7.1, U1.2 (-)
- new net: R17.2, R18.1, R7.2
- new net: C1.2, C5.2, R19.2, R5.2, U1.6
- new net: R12.1, R13.2, U4.2 (-)
- new net: C5.1, R11.1, U4.3 (+)
- new net: R17.1, R9.1
- new net: R19.1, R20.2, R8.2
- new net B+: IC1.6 (-IN_B)
- new net C+: IC1.9 (-IN_C)
- new net VCC: U1.7 (V+), U2.7 (V+), U3.7 (V+), U4.7 (V+), V2.1
- new net VEE: U1.4 (V-), U2.4 (V-), U3.4 (V-), U4.4 (V-), V1.2
Other:
- moved on the sheet: C6, R1, RV1A, RV1B, RV3, RV4

Commit message: started main schematic
Parts:
- removed C2, C3: 100uF, symbol Device:C
- removed C6, C7: 10u, symbol Device:C
- removed R14: 100, Resistor_THT:R_Axial_DIN0207_L6.3mm_D2.5mm_P10.16mm_Horizontal, symbol Device:R
- removed R15, R18, R19, R22: 10k, Resistor_THT:R_Axial_DIN0207_L6.3mm_D2.5mm_P10.16mm_Horizontal, symbol Device:R
- removed R16, R17, R20, R21: 10, Resistor_THT:R_Axial_DIN0207_L6.3mm_D2.5mm_P10.16mm_Horizontal, symbol Device:R
- removed U1, U2, U3, U4: OPA1641, OPA1641:OPA1641, symbol Amplifier_Operational:OPA1641
- removed V1, V2: 16, symbol Simulation_SPICE:VDC
- removed V3: VSIN, symbol Simulation_SPICE:VSIN
Connections:
- net 0 is gone; now on net GND: R1.2, R11.2
- net B+ is gone; now on net B-: IC1.6 (-IN_B)
- net C+ is gone; now on net C-: IC1.9 (-IN_C)
- net A+: now also R5.1, R6.1, RV3.1
- net A-: now also R2.1, R3.2, R4.2
- net Ao: now also R3.1, RV1.1
- net B-: now also C1.1, R7.1; no longer IC1.5 (+IN_B)
- net Bo: now also C1.2, C5.2, R5.2, RV1.4
- net C-: now also C4.1, R8.1; no longer IC1.10 (+IN_C)
- net Co: now also C4.2, R4.1
- net D+: now also C5.1, R11.1
- net D-: now also R12.1, R13.2
- net Do: now also R12.2, RV4.3
- net Input: now also R13.1, RV4.1
- net VCC: now also IC1.4 (V+)
- net VEE: now also IC1.11 (V-)
- net at RV1.5: now also R8.2
- net at RV1.6: now also R10.1
- net at RV1.2: now also R7.2
- net at RV1.3: now also R9.1
- net at R6.2: now also RV4.2
- net at R1.1: now also RV3.2
- net at R2.2: now also RV3.3
- net GND: now reaches R9.2
- net GND: now also IC1.10 (+IN_C), IC1.5 (+IN_B), R10.2
Other:
- moved on the sheet: R2
