File: Low_Pass_Filter/LPF/LPF.kicad_sch (KiCad schematic)
At the start: 7 parts, among them U1 OPA1641

Commit message: started main schematic
Connections:
- net at R4.2, U1.6: now also C1.2; no longer C1.1
- net at RV1.2: now also C1.1; no longer C1.2
Other:
- moved on the sheet: C1
Changed lines of the file:
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@@
 	(wire
 		(pts
-			(xy 55.88 15.24) (xy 96.52 15.24)
-		)
-		(stroke
-			(width 0)
-			(type default)
-		)
-	)
-	(wire
-		(pts
-			(xy 55.88 22.86) (xy 55.88 29.21)
+			(xy 55.88 20.32) (xy 55.88 29.21)
 		)
 		(stroke
@@
 	(wire
 		(pts
-			(xy 96.52 15.24) (xy 96.52 35.56)
-		)
-		(stroke
-			(width 0)
-			(type default)
-		)
-	)
-	(wire
-		(pts
 			(xy 74.93 33.02) (xy 81.28 33.02)
 		)
@@
 	(wire
 		(pts
+			(xy 55.88 20.32) (xy 68.58 20.32)
+		)
+		(stroke
+			(width 0)
+			(type default)
+		)
+	)
+	(wire
+		(pts
 			(xy 96.52 35.56) (xy 96.52 48.26)
 		)
@@
 		(pts
 			(xy 96.52 35.56) (xy 101.6 35.56)
+		)
+		(stroke
+			(width 0)
+			(type default)
+		)
+	)
+	(wire
+		(pts
+			(xy 96.52 20.32) (xy 96.52 35.56)
+		)
+		(stroke
+			(width 0)
+			(type default)
+		)
+	)
+	(wire
+		(pts
+			(xy 76.2 20.32) (xy 96.52 20.32)
 		)
 		(stroke
@@
 	(symbol
 		(lib_id "Device:C")
-		(at 55.88 19.05 0)
+		(at 72.39 20.32 90)
 		(unit 1)
 		(exclude_from_sim no)
@@
 		(fields_autoplaced yes)
 		(property "Reference" "C1"
-			(at 59.69 17.7799 0)
-			(effects
-				(font
-					(size 1.27 1.27)
-				)
-				(justify left)
+			(at 72.39 12.7 90)
+			(effects
+				(font
+					(size 1.27 1.27)
+				)
 			)
 		)
 		(property "Value" "20n"
-			(at 59.69 20.3199 0)
-			(effects
-				(font
-					(size 1.27 1.27)
-				)
-				(justify left)
+			(at 72.39 15.24 90)
+			(effects
+				(font
+					(size 1.27 1.27)
+				)
 			)
 		)
 		(property "Footprint" ""
-			(at 56.8452 22.86 0)
+			(at 76.2 19.3548 0)
 			(effects
 				(font
@@
 		)
 		(property "Datasheet" "~"
-			(at 55.88 19.05 0)
+			(at 72.39 20.32 0)
 			(effects
 				(font
@@
 		)
 		(property "Description" "Unpolarized capacitor"
-			(at 55.88 19.05 0)
+			(at 72.39 20.32 0)
 			(effects
 				(font
@@
 		)
 		(instances
-			(project ""
+			(project "LPF"
 				(path "/1e068942-4d60-4b61-a79e-d88caf00654c"
 					(reference "C1")
@@
 		(dnp no)
 		(property "Reference" "U1"
-			(at 91.948 28.702 0)
+			(at 89.662 31.496 0)
 			(effects
 				(font
@@
 		)
 		(property "Value" "OPA1641"
-			(at 91.948 31.242 0)
-			(effects
-				(font
+			(at 88.392 35.56 0)
+			(effects
+				(font
