File: Combined_EQ/Combined_EQ.kicad_sch (KiCad schematic)
At the start: 115 parts, among them IC1 INA137PA, IC2 OPA1644AIPWR, IC3 OPA1644AIPWR, IC4 OPA1644AIPWR, IC5 OPA1644AIPWR, IC6 DRV134PA, J1 EDA 306, SW1 SW_Slide_DPDT

Commit message: started on pcb
need to footprint for the capacitors
Parts:
- R1, R2, R3, R4, R45, R47, R53, R54: footprint (none) -> Resistor_THT:R_Axial_DIN0207_L6.3mm_D2.5mm_P10.16mm_Horizontal
- R10, R11, R12, R13, R40, R41, R42, R43, R44, R46, R48, R49, R5, R50, R51, R52, R55, R6, R7, R8, R9: footprint (none) -> R_Axial_DIN0207_L6.3mm_D2.5mm_P10.16mm_Horizontal
- RV1, RV4, RV6, RV9: footprint (none) -> Potentiometer_THT:Potentiometer_Alps_RK097_Dual_Horizontal
- RV10, RV2, RV3, RV5, RV7, RV8: footprint (none) -> Potentiometer_THT:Potentiometer_Alps_RK097_Single_Horizontal
- SW1: footprint (none) -> Button_Switch_THT:SW_CK_JS202011CQN_DPDT_Straight
