File: Combined_EQ/Combined_EQ.kicad_sch (KiCad schematic)
At the start: 115 parts, among them IC1 INA137PA, IC2 OPA1644AIPWR, IC3 OPA1644AIPWR, IC4 OPA1644AIPWR, IC5 OPA1644AIPWR, IC6 DRV134PA, J1 EDA 306, SW1 SW_Slide_DPDT

Commit message: half done pcb
Parts:
- added C39, C42: 2.2n, Capacitor_THT:C_Disc_D5.0mm_W2.5mm_P5.00mm, symbol Device:C
- added C40: 470p, Capacitor_THT:C_Disc_D5.0mm_W2.5mm_P5.00mm, symbol Device:C
- added C41, C44: 100p, Capacitor_THT:C_Disc_D5.0mm_W2.5mm_P5.00mm, symbol Device:C
- added C43, C46, C47: 10n, Capacitor_THT:C_Disc_D5.0mm_W2.5mm_P5.00mm, symbol Device:C
- added H1, H2, H3, H4: MountingHole, MountingHole:MountingHole_3.2mm_M3, symbol Mechanical:MountingHole
- C1, C11, C12, C13, C14, C15, C16, C17, C18, C19, C20, C21, C22, C23, C25, C26, C28, C29, C30, C31, C32, C33, C34, C35, C36, C37, C38, C5: footprint (none) -> Capacitor_THT:C_Disc_D5.0mm_W2.5mm_P5.00mm
- C10, C4: footprint (none) -> Capacitor_THT:C_Radial_D8.0mm_H7.0mm_P3.50mm
- C2, C7: footprint (none) -> Capacitor_THT:C_Rect_L4.0mm_W2.5mm_P2.50mm
- C24, C27: value 20n -> 10n; footprint (none) -> Capacitor_THT:C_Disc_D5.0mm_W2.5mm_P5.00mm
- C3, C6: value 2.3n -> 2.2n; footprint (none) -> Capacitor_THT:C_Disc_D5.0mm_W2.5mm_P5.00mm
- C8: value 12.7nF -> 10n; footprint (none) -> Capacitor_THT:C_Disc_D5.0mm_W2.5mm_P5.00mm
- C9: value 12.7nF -> 470p; footprint (none) -> Capacitor_THT:C_Disc_D5.0mm_W2.5mm_P5.00mm
Connections:
- net +16V: now also C15.2, C21.2, IC4.4 (V+); no longer C13.1
- net +IN+4: no longer SW1.4 (A)
- net -16V: now also C13.2, C14.2, C16.2, C22.2, C30.2, C31.2; no longer C14.1, C15.1, C16.1, C21.1, C22.1, C30.1, C31.1, IC4.4 (V+)
- net -IN+4: no longer SW1.3 (C)
- net B-: now also C39.1, C40.1
- net Bo: now also C39.2, C40.2
- net C-: now also C42.1, C43.1
- net Co: now also C42.2, C43.2
- net F-: now also C41.1
- net Fo: now also C41.2
- net G-: now also C44.1
- net GND: now also C13.1, C14.1, C15.1, C16.1, C21.1, C22.1, C30.1, C31.1, C46.2, C47.2; no longer C13.2, C14.2, C15.2, C16.2, C21.2, C22.2, C27.1, C30.2, C31.2
- net Go: now also C44.2
- net K+: now also C46.1, C47.1; no longer C27.2
- net Ko: now also C27.1
- net -IN: now reaches FB1.2, R1.1
- net -IN: now also SW1.3 (C)
- net at C24.2, R9.1, RV1.3: now also C27.2
- net +IN: now reaches FB2.2, R3.1
- net +IN: now also SW1.4 (A)

Commit message: more progress
Parts:
- added J2, J3: Conn_01x24_Pin, symbol Connector:Conn_01x24_Pin
Other:
- moved on the sheet: H1, H2, H3, H4

Commit message: components placed
need to wire up
Parts:
- removed IC2, IC3, IC4, IC5: OPA1644AIPWR, OPA1644:SOP65P640X120-14N, symbol OPA1644AIPWR:OPA1644AIPWR
- removed J2, J3: Conn_01x24_Pin, symbol Connector:Conn_01x24_Pin
- added C45, C48: 100n, Capacitor_THT:C_Disc_D5.0mm_W2.5mm_P5.00mm, symbol Device:C
- added IC2, IC3, IC4, IC8: OPA1644AID, OPA1644AID:SOIC127P600X175-14N, symbol OPA1644AID:OPA1644AID
- added J2: Conn_01x17_Pin, Connector_PinHeader_2.54mm:PinHeader_1x17_P2.54mm_Vertical, symbol Connector:Conn_01x17_Pin
- added J3: Conn_01x17_Pin, Connector_PinSocket_2.54mm:PinSocket_1x17_P2.54mm_Vertical, symbol Connector:Conn_01x17_Pin
- added U1: OPA1641, OPA1641AID:SOIC127P600X175-8N, symbol Amplifier_Operational:OPA1641
Connections:
- net +16V: now also C13.2, C30.2, C45.2, IC2.4 (V+), IC3.4 (V+), IC4.4 (V+), IC8.4 (V+), U1.7 (V+)
- net -16V: now also C48.2, IC2.11 (V-), IC3.11 (V-), IC4.11 (V-), IC8.11 (V-), U1.4 (V-); no longer C13.2, C30.2
- net A+: now also IC3.3 (+_IN_A)
- net A-: now also IC3.2 (-IN_A)
- net Ao: now also IC3.1 (OUT_A), J3.11 (Pin_11); no longer RV9.1
- net B-: now also IC3.6 (-_IN_B)
- net Bo: now also IC3.7 (OUT_B), J3.9 (Pin_9); no longer RV9.4
- net C-: now also IC3.9 (-IN_C)
- net Co: now also IC3.8 (OUT_C)
- net D+: now also IC3.12 (+IN_D)
- net D-: now also IC3.13 (-_IN_D)
- net Do: now also IC3.14 (OUT_D)
- net E+: now also IC2.3 (+_IN_A)
- net E-: now also IC2.2 (-IN_A)
- net Eo: now also IC2.1 (OUT_A), J3.6 (Pin_6); no longer RV6.1
- net F-: now also IC2.6 (-_IN_B)
- net Fo: now also IC2.7 (OUT_B), J3.5 (Pin_5); no longer RV6.4
- net G-: now also IC2.13 (-_IN_D)
- net GND: now also C45.1, C48.1, IC2.12 (+IN_D), IC2.5 (+IN_B), IC3.10 (+_IN_C), IC3.5 (+IN_B), IC8.10 (+_IN_C), IC8.12 (+IN_D), IC8.3 (+_IN_A), IC8.5 (+IN_B), J3.15 (Pin_15); no longer C46.2, C47.2, R21.2, R25.2, R34.2, R37.2, RV4.3
- net Go: now also IC2.14 (OUT_D)
- net H+: now also IC2.10 (+_IN_C)
- net H-: now also IC2.9 (-IN_C)
- net Ho: now also IC2.8 (OUT_C)
- net J+: now also IC4.5 (+IN_B)
- net J-: now also IC4.6 (-_IN_B), IC4.7 (OUT_B)
- net K+: now also IC4.12 (+IN_D), J3.12 (Pin_12); no longer C46.1, C47.1, RV1.6
- net K-: now also IC4.13 (-_IN_D)
- net Ko: now also IC4.14 (OUT_D), J3.14 (Pin_14); no longer C24.1, C27.1
- net L+: now also IC4.10 (+_IN_C), J3.3 (Pin_3); no longer R42.1
- net L-: now also IC4.9 (-IN_C)
- net Lo: now also IC4.8 (OUT_C), J3.1 (Pin_1); no longer RV4.6
- net M-: now also IC8.2 (-IN_A)
- net Mo: now also IC8.1 (OUT_A)
- net N-: now also IC8.6 (-_IN_B)
- net No: now also IC8.7 (OUT_B)
- net O-: now also IC8.13 (-_IN_D)
- net Oo: now also IC8.14 (OUT_D)
- net P-: now also IC8.9 (-IN_C)
- net Po: now also IC8.8 (OUT_C)
- net T13: now reaches RV1.1, RV1.2
- net T13: now also J2.13 (Pin_13); no longer R8.2
- net B4: now reaches R26.2
- net B4: now also J3.4 (Pin_4); no longer RV6.5
- net B8: now reaches R38.2
- net B8: now also J3.8 (Pin_8); no longer RV9.5
- net B2: now reaches C25.2, C26.1
- net B2: now also J3.2 (Pin_2); no longer R40.1
- net B7: now reaches R24.2
- net B7: now also J3.7 (Pin_7); no longer RV6.2
- net B10: now reaches R36.2
- net B10: now also J3.10 (Pin_10); no longer RV9.2
- net I+: no longer names the net of IC1.5 (SENSE), IC1.6 (OUTPUT)
- net I+: now also U1.3 (+)
- net I-: no longer names the net of R29.1, RV8.1
- net I-: now also U1.2 (-), U1.6
- new net B13: J3.13 (Pin_13), R8.2
- new net T1: J2.1 (Pin_1), RV4.6
- new net T10: J2.10 (Pin_10), RV9.2
- new net T11: J2.11 (Pin_11), RV9.1
- new net T12: C46.1, C47.1, J2.12 (Pin_12), RV1.6
- new net T14: C24.1, C27.1, J2.14 (Pin_14)
- new net T15: C46.2, C47.2, J2.15 (Pin_15), R21.2, R25.2, R34.2, R37.2, RV4.3
- new net T2: J2.2 (Pin_2), R40.1
- new net T3: J2.3 (Pin_3), R42.1
- new net T4: J2.4 (Pin_4), RV6.5
- new net T5: J2.5 (Pin_5), RV6.4
- new net T6: J2.6 (Pin_6), RV6.1
- new net T7: J2.7 (Pin_7), RV6.2
- new net T8: J2.8 (Pin_8), RV9.5
- new net T9: J2.9 (Pin_9), RV9.4
- no-connect marks 6 -> 13
Other:
- note added: "BOTTOM BOARD"
- note added: "TOP BOARD"

Commit message: finalised and ordered
Parts:
- J3: footprint Connector_PinSocket_2.54mm:PinSocket_1x17_P2.54mm_Vertical -> Connector_PinHeader_2.54mm:PinHeader_1x17_P2.54mm_Vertical
Connections:
- net T15 is gone; now on net GND: C46.2, C47.2, J2.15 (Pin_15), R21.2, R25.2, R34.2, R37.2, RV4.3
