File: Combined_EQ/Combined_EQ.kicad_pcb (KiCad board)
At the start: 4 copper layers, 167.3 x 105 mm, 133 parts, among them IC1 INA137PA, IC2 OPA1644AID, IC3 OPA1644AID, IC4 OPA1644AID, IC6 DRV134PA, IC8 OPA1644AID, J1 EDA 306, J2 Conn_01x17_Pin, J3 Conn_01x17_Pin, SW1 SW_Slide_DPDT, U1 OPA1641

Commit message: finalised and ordered
Parts:
- G***: value LOGO -> (none)
- J3: footprint Connector_PinSocket_2.54mm:PinSocket_1x17_P2.54mm_Vertical -> Connector_PinHeader_2.54mm:PinHeader_1x17_P2.54mm_Vertical
- moved R2 16.6 mm to (157.7, 81.7), turned to 90 degrees
- moved C43 7.84 mm to (94.9, 88.2), turned to 180 degrees
- moved C9 7.82 mm to (94.9, 93.2), turned to 180 degrees
- moved C42 7.82 mm to (94.9, 83.5), turned to 180 degrees
- moved R4 7.49 mm to (157.7, 58.7), turned to -90 degrees
- moved R5 7.21 mm to (187.9, 133.9)
- moved C45 5.27 mm to (131.7, 83.0)
- moved C48 5.27 mm to (129.2, 67.8)
- moved U1 5.27 mm to (131.7, 73.5)
- moved C22 4.76 mm to (129.7, 130.5), turned to 180 degrees
- moved R32 4.39 mm to (119.7, 72.0)
- moved C7 4.31 mm to (110.4, 78.0)
- moved C11 3.51 mm to (147.9, 57.5)
- moved C12 3.51 mm to (143.2, 84.0)
- moved C37 3.51 mm to (142.7, 57.5)
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Connections:
- C11 pad 1: B+ -> GND
- C12 pad 1: B+ -> GND
- C13 pad 1: B+ -> GND
- C14 pad 1: B+ -> GND
- C15 pad 1: B+ -> GND
- C16 pad 1: B+ -> GND
- C17 pad 2: B+ -> GND
- C18 pad 2: B+ -> GND
- C19 pad 1: B+ -> GND
- C20 pad 1: B+ -> GND
- C21 pad 1: B+ -> GND
- C22 pad 1: B+ -> GND
- C30 pad 1: B+ -> GND
- C31 pad 1: B+ -> GND
- C32 pad 2: B+ -> GND
- C34 pad 2: B+ -> GND
- C35 pad 2: B+ -> GND
- C36 pad 1: B+ -> GND
- C37 pad 1: B+ -> GND
- C38 pad 1: B+ -> GND
- C45 pad 1: B+ -> GND
- C46 pad 2: /T15 -> GND
- C47 pad 2: /T15 -> GND
- C48 pad 1: B+ -> GND
- IC1 pad 1: B+ -> GND
- IC2 pad 12: B+ -> GND
- IC2 pad 5: B+ -> GND
- IC3 pad 10: B+ -> GND
- IC3 pad 5: B+ -> GND
- IC6 pad 3: B+ -> GND
- IC8 pad 10: B+ -> GND
- IC8 pad 12: B+ -> GND
- IC8 pad 3: B+ -> GND
- IC8 pad 5: B+ -> GND
- J1 pad 13: B+ -> GND
- J1 pad 5: B+ -> GND
- J2 pad 15: /T15 -> GND
- J3 pad 15: B+ -> GND
- R10 pad 2: B+ -> GND
- R13 pad 2: B+ -> GND
- R14 pad 2: B+ -> GND
- R2 pad 1: B+ -> GND
- R20 pad 2: B+ -> GND
- R21 pad 2: /T15 -> GND
- R25 pad 2: /T15 -> GND
- R27 pad 2: B+ -> GND
- R33 pad 2: B+ -> GND
- R34 pad 2: /T15 -> GND
- R37 pad 2: /T15 -> GND
- R4 pad 1: B+ -> GND
- R41 pad 2: B+ -> GND
- R7 pad 1: B+ -> GND
- RV4 pad 3: /T15 -> GND
Routing:
- net -16V: track 0.00 -> 262.1 mm, vias 0 -> 3
- net +16V: track 0.00 -> 246.7 mm, vias 0 -> 3
- net M-: track 0.00 -> 144.3 mm, vias 0 -> 1
- net N-: track 0.00 -> 133.3 mm, vias 0 -> 1
- net Net-(R48-Pad1): track 0.00 -> 126.6 mm
- net Lo: track 0.00 -> 117.8 mm, vias 0 -> 3
- net Net-(R46-Pad1): track 0.00 -> 101.7 mm, vias 0 -> 2
- net Fo: track 0.00 -> 96.1 mm, vias 0 -> 4
- net Do: track 0.00 -> 89.8 mm, vias 0 -> 2
- net Net-(R47-Pad2): track 0.00 -> 88.5 mm, vias 0 -> 1
- net Net-(R45-Pad2): track 0.00 -> 88.1 mm, vias 0 -> 1
- net /B2: track 0.00 -> 85.0 mm, vias 0 -> 3
- net Net-(U1--): track 0.00 -> 83.2 mm, vias 0 -> 2
- net L+: track 0.00 -> 73.3 mm, vias 0 -> 1
- net E+: track 0.00 -> 70.6 mm, vias 0 -> 3
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- added copper zone on In1.Cu, net GND
